Commit message: readme.md update

File: ros2_ws/src/example_1/description/urdf/rrbot_description.urdf.xacro (robot description, xacro)
@@ -84,5 +84,5 @@
     <parent link="${prefix}link1"/>
     <child link="${prefix}link2"/>
-    <axis xyz="0 1 0"/>
+    <axis xyz="0 -1 0"/>
     <dynamics damping="0.7"/>
     <limit lower="${-1.75}" upper="${1.75}" effort="1.0" velocity="1.0"/>
@@ -117,5 +117,5 @@
     <child link="${prefix}link3"/>
     <origin xyz="0 ${width} ${height2 - axel_offset*2}" rpy="0 0 0"/>
-    <axis xyz="0 1 0"/>
+    <axis xyz="0 -1 0"/>
     <dynamics damping="0.7"/>
     <limit lower="${-1.75}" upper="${1.75}" effort="1.0" velocity="1.0"/>
